Commit message: Added simulation results

File: src/p3dx_gazebo/xacro/p3dx/pioneer3dx.sick.xacro (robot description, xacro)
@@ -15,5 +15,6 @@
 	<xacro:sick_tim310 name="laser" ros_topic="laser/scan" rpy="${pi} 0 0"/>
 	<joint name="base_laser_joint" type="fixed">
-		<origin xyz="0.16 0 0.1" rpy="0 0 0"/>
+		<!-- origin xyz="0.16 0 0.1" rpy="0 0 0"/ -->
+		<origin xyz="0.17 0 0.05" rpy="0 0 0"/>
 		<axis xzy="0 1 0"/>
 		<parent link="chassis"/>

File: src/sick_tim/urdf/sick_tim.urdf.xacro (robot description, xacro)
@@ -53,5 +53,5 @@
       </inertial>
     </link>
-    <xacro:sick_tim_laser_gazebo_v0 name="${name}" link="${name}" ros_topic="${ros_topic}" update_rate="15.0" min_angle="-2.357" max_angle="2.357" min_range="${min_range}" max_range="${max_range}"/>
+    <xacro:sick_tim_laser_gazebo_v0 name="${name}" link="${name}" ros_topic="${ros_topic}" update_rate="15.0" min_angle="-2.0" max_angle="2.0" min_range="${min_range}" max_range="${max_range}"/>
   </xacro:macro>
   <xacro:macro name="sick_tim_laser_gazebo_v0" params="name link ros_topic update_rate min_angle max_angle min_range max_range">
