Commit message: added velodyne to real robot

File: src/amr-ros-config/description/urdf/pioneer3dx.urdf (robot description, URDF)
Before this commit: robot pioneer3dx, 14 links, 13 joints
Links:
- added link velodyne, mass 0.1; visual mesh filename=package://velodyne_description/meshes/VLP16_scan.dae
- added link velodyne_base_link, mass 0.1; collision cylinder length=0.0717 radius=0.0516; visual mesh filename=package://velodyne_description/meshes/VLP16_base_1.dae
Joints:
- added joint velodyne_base_mount_joint: type fixed, parent base_link, child velodyne_base_link, origin xyz=0 0 0.4 rpy=0 0 0
- added joint velodyne_base_scan_joint: type fixed, parent velodyne_base_link, child velodyne, origin xyz=0 0 0.0377 rpy=0 0 0

File: src/amr-ros-config/description/urdf/pioneer3dx.urdf.xacro (robot description, xacro)
@@ -8,13 +8,17 @@
   <!--<include filename="$(find amr_robots_description)/urdf/materials.xacro"/>-->
   <xacro:include filename="$(find amr_robots_description)/urdf/pioneer3dx_wheel.xacro"/>
-<!-- Laser -->
-	<xacro:include filename="$(find sick_tim)/urdf/sick_tim.urdf.xacro"/>
-	<xacro:sick_tim310 name="laser" ros_topic="scan" rpy="${pi} 0 0" />
-	<joint name="base_laser_joint" type="fixed">
-		<origin xyz="0.16 0 0.1" rpy="0 0 0"/>
-		<axis xzy="0 1 0"/>
-		<parent link="base_link"/>
-		<child link="laser_mount_link"/>
-	</joint>
+  <!-- Laser -->
+  <xacro:include filename="$(find sick_tim)/urdf/sick_tim.urdf.xacro"/>
+  <xacro:sick_tim310 name="laser" ros_topic="scan" rpy="${pi} 0 0" />
+  <joint name="base_laser_joint" type="fixed">
+    <origin xyz="0.16 0 0.1" rpy="0 0 0"/>
+    <axis xzy="0 1 0"/>
+    <parent link="base_link"/>
+    <child link="laser_mount_link"/>
+  </joint>
+  <xacro:include filename="$(find p3dx_gazebo)/xacro/laser/VLP-16.urdf.xacro"/>
+  <VLP-16 parent="base_link" name="velodyne" topic="/velodyne_points">
+    <origin xyz="0 0 0.4" rpy="0 0 0" />
+  </VLP-16>
 <!-- Camera -->
 <joint name="$base_link_camera_joint" type="fixed">
